File: TinyBoard84100.sch (KiCad schematic (older format))
At the start: 14 parts

Commit message: test
Other:
- moved on the sheet: C?, P?, U?
Changed lines of the file:
@@
 $EndDescr
-$Comp
-L ATTINY841 U?
-U 1 1 5AD23C06
-P 4200 3600
-F 0 "U?" H 3150 4400 60  0000 C CNN
-F 1 "ATTINY841" H 3300 2800 60  0000 C CNN
-F 2 "" H 5250 3000 60  0000 C CNN
-F 3 "" H 5250 3000 60  0000 C CNN
-	1    4200 3600
-	1    0    0    -1
-$EndComp
 $Comp
 L SW_PUSH SW?
@@
 L CONN_01X02 P?
 U 1 1 5AD23D2C
-P 7400 3300
-F 0 "P?" H 7400 3450 50  0000 C CNN
-F 1 "CONN_01X02" V 7500 3300 50  0000 C CNN
-F 2 "" H 7400 3300 50  0000 C CNN
-F 3 "" H 7400 3300 50  0000 C CNN
-	1    7400 3300
-	1    0    0    -1
+P 1300 1600
+F 0 "P?" H 1300 1750 50  0000 C CNN
+F 1 "CONN_01X02" V 1400 1600 50  0000 C CNN
+F 2 "" H 1300 1600 50  0000 C CNN
+F 3 "" H 1300 1600 50  0000 C CNN
+	1    1300 1600
+	-1   0    0    -1
 $EndComp
 $Comp
@@
 L C C?
 U 1 1 5AD23DAF
-P 8450 3150
-F 0 "C?" H 8450 3250 40  0000 L CNN
-F 1 "C" H 8456 3065 40  0000 L CNN
-F 2 "" H 8488 3000 30  0000 C CNN
-F 3 "" H 8450 3150 60  0000 C CNN
-	1    8450 3150
+P 2750 1950
+F 0 "C?" H 2750 2050 40  0000 L CNN
+F 1 "C" H 2756 1865 40  0000 L CNN
+F 2 "" H 2788 1800 30  0000 C CNN
+F 3 "" H 2750 1950 60  0000 C CNN
+	1    2750 1950
 	1    0    0    -1
 $EndComp
@@
 $EndComp
 $Comp
-L 78L05 U?
-U 1 1 5AD23F10
-P 6450 1750
-F 0 "U?" H 6550 1650 60  0000 C CNN
-F 1 "78L05" H 6450 2000 60  0000 C CNN
-F 2 "" H 6350 1850 60  0000 C CNN
-F 3 "" H 6350 1850 60  0000 C CNN
-	1    6450 1750
-	1    0    0    -1
-$EndComp
-$Comp
 L CONN_01X07 P?
 U 1 1 5AD23FFE
@@
 $EndComp
 $Comp
+L PWR_FLAG #FLG?
+U 1 1 5AD2529F
+P 1900 1400
+F 0 "#FLG?" H 1900 1495 50  0001 C CNN
+F 1 "PWR_FLAG" H 1900 1580 50  0000 C CNN
+F 2 "" H 1900 1400 50  0000 C CNN
+F 3 "" H 1900 1400 50  0000 C CNN
+	1    1900 1400
+	1    0    0    -1
+$EndComp
+$Comp
+L PWR_FLAG #FLG?
+U 1 1 5AD252DB
+P 1900 1800
+F 0 "#FLG?" H 1900 1895 50  0001 C CNN
+F 1 "PWR_FLAG" H 1900 1980 50  0000 C CNN
+F 2 "" H 1900 1800 50  0000 C CNN
+F 3 "" H 1900 1800 50  0000 C CNN
+	1    1900 1800
+	1    0    0    1
+$EndComp
+$Comp
 L GND #PWR?
-U 1 1 5AD23EE5
-P 4350 1600
-F 0 "#PWR?" H 4350 1350 50  0001 C CNN
-F 1 "GND" H 4350 1450 50  0000 C CNN
-F 2 "" H 4350 1600 50  0000 C CNN
-F 3 "" H 4350 1600 50  0000 C CNN
-	1    4350 1600
+U 1 1 5AD25364
+P 2400 1800
+F 0 "#PWR?" H 2400 1550 50  0001 C CNN
+F 1 "GND" H 2400 1650 50  0000 C CNN
+F 2 "" H 2400 1800 50  0000 C CNN
+F 3 "" H 2400 1800 50  0000 C CNN
+	1    2400 1800
 	1    0    0    -1
 $EndComp
 $Comp
 L +5V #PWR?
-U 1 1 5AD23F23
-P 3750 1550
-F 0 "#PWR?" H 3750 1400 50  0001 C CNN
-F 1 "+5V" H 3750 1690 50  0000 C CNN
-F 2 "" H 3750 1550 50  0000 C CNN
-F 3 "" H 3750 1550 50  0000 C CNN
-	1    3750 1550
+U 1 1 5AD253A2
+P 2400 1400
+F 0 "#PWR?" H 2400 1250 50  0001 C CNN
+F 1 "+5V" H 2400 1540 50  0000 C CNN
+F 2 "" H 2400 1400 50  0000 C CNN
+F 3 "" H 2400 1400 50  0000 C CNN
+	1    2400 1400
 	1    0    0    -1
 $EndComp
+$Comp
+L 78L05 U?
+U 1 1 5AD23F10
+P 3150 1250
+F 0 "U?" H 3250 1150 60  0000 C CNN
+F 1 "78L05" H 3150 1500 60  0000 C CNN
+F 2 "" H 3050 1350 60  0000 C CNN
+F 3 "" H 3050 1350 60  0000 C CNN
+	1    3150 1250
+	1    0    0    -1
+$EndComp
+$Comp
+L ATTINY841 U?
+U 1 1 5AD23C06
+P 4100 3800
+F 0 "U?" H 3050 4600 60  0000 C CNN
+F 1 "ATTINY841" H 3200 3000 60  0000 C CNN
+F 2 "" H 5150 3200 60  0000 C CNN
+F 3 "" H 5150 3200 60  0000 C CNN
+	1    4100 3800
+	1    0    0    -1
+$EndComp

Commit message: Wiring ideas
Connections:
- net labels added: MISO, MOSI, PA0, PA1, PA2, PA3, PA4, PA5, PA6, PA7, PB0, PB1, PB2, PB3, SCK, ~RST
- wire segments 0 -> 32
Other:
- moved on the sheet: C?, D?, P?, R?, SW?, U?

Commit message: Wires and lables
Connections:
- wire segments 32 -> 46
Other:
- moved on the sheet: P?
Changed lines of the file:
@@
 L CONN_01X07 P?
 U 1 1 5AD23FFE
-P 7350 5300
-F 0 "P?" H 7350 5700 50  0000 C CNN
-F 1 "CONN_01X07" V 7450 5300 50  0000 C CNN
-F 2 "" H 7350 5300 50  0000 C CNN
-F 3 "" H 7350 5300 50  0000 C CNN
-	1    7350 5300
-	1    0    0    -1
+P 2950 5800
+F 0 "P?" H 2950 6200 50  0000 C CNN
+F 1 "CONN_01X07" V 3050 5800 50  0000 C CNN
+F 2 "" H 2950 5800 50  0000 C CNN
+F 3 "" H 2950 5800 50  0000 C CNN
+	1    2950 5800
+	-1   0    0    -1
 $EndComp
 $Comp
 L CONN_01X07 P?
 U 1 1 5AD240B6
-P 8100 5300
-F 0 "P?" H 8100 5700 50  0000 C CNN
-F 1 "CONN_01X07" V 8200 5300 50  0000 C CNN
-F 2 "" H 8100 5300 50  0000 C CNN
-F 3 "" H 8100 5300 50  0000 C CNN
-	1    8100 5300
+P 5250 5800
+F 0 "P?" H 5250 6200 50  0000 C CNN
+F 1 "CONN_01X07" V 5350 5800 50  0000 C CNN
+F 2 "" H 5250 5800 50  0000 C CNN
+F 3 "" H 5250 5800 50  0000 C CNN
+	1    5250 5800
 	1    0    0    -1
 $EndComp
@@
 	1    0    0    -1
 $EndComp
-Wire Wire Line
-	5600 3100 6200 3100
-Wire Wire Line
-	5600 3300 6200 3300
-Wire Wire Line
-	5600 3500 6200 3500
-Wire Wire Line
-	5600 3700 6200 3700
-Wire Wire Line
-	5600 3900 6200 3900
-Wire Wire Line
-	5600 4100 6200 4100
-Wire Wire Line
-	5600 4300 6200 4300
-Wire Wire Line
-	5600 4500 6200 4500
-Wire Wire Line
-	2600 3200 2100 3200
-Wire Wire Line
-	2600 3600 2100 3600
-Wire Wire Line
-	2600 4000 2100 4000
-Wire Wire Line
-	1900 4400 2600 4400
 $Comp
 L GND #PWR?
@@
 Wire Wire Line
 	1500 4250 1500 4400
-Text Label 2100 3200 0    60   ~ 0
+Text Label 2250 3200 0    60   ~ 0
 PB0
-Text Label 2100 3600 0    60   ~ 0
+Text Label 2250 3600 0    60   ~ 0
 PB1
-Text Label 2100 4000 0    60   ~ 0
+Text Label 2250 4000 0    60   ~ 0
 PB2
-Text Label 2100 4400 0    60   ~ 0
+Text Label 2250 4400 0    60   ~ 0
 PB3
-Text Label 5800 3100 0    60   ~ 0
+Text Label 5950 3100 2    60   ~ 0
 PA0
-Text Label 5800 3300 0    60   ~ 0
+Text Label 5950 3300 2    60   ~ 0
 PA1
-Text Label 5800 3500 0    60   ~ 0
+Text Label 5950 3500 2    60   ~ 0
 PA2
-Text Label 5800 3700 0    60   ~ 0
+Text Label 5950 3700 2    60   ~ 0
 PA3
-Text Label 5800 3900 0    60   ~ 0
+Text Label 5950 3900 2    60   ~ 0
 PA4
-Text Label 5800 4100 0    60   ~ 0
+Text Label 5950 4100 2    60   ~ 0
 PA5
-Text Label 5800 4300 0    60   ~ 0
+Text Label 5950 4300 2    60   ~ 0
 PA6
-Text Label 5800 4500 0    60   ~ 0
+Text Label 5950 4500 2    60   ~ 0
 PA7
 Wire Wire Line
@@
 Text Label 7500 3650 0    60   ~ 0
 ~RST
-Text Label 8350 3400 0    60   ~ 0
+Text Label 8550 3400 2    60   ~ 0
 MOSI
 Wire Wire Line
@@
 	1    0    0    -1
 $EndComp
+Wire Wire Line
+	3150 5800 3400 5800
+Wire Wire Line
+	3150 5700 3400 5700
+Wire Wire Line
+	3150 5600 3400 5600
+Wire Wire Line
+	3150 5500 3400 5500
+Wire Wire Line
+	3150 5900 3400 5900
+Wire Wire Line
+	3150 6000 3400 6000
+Wire Wire Line
+	3150 6100 3400 6100
+Wire Wire Line
+	5050 5500 4800 5500
+Wire Wire Line
+	5050 5600 4800 5600
+Wire Wire Line
+	5050 5700 4800 5700
+Wire Wire Line
+	5050 5800 4800 5800
+Wire Wire Line
+	5050 5900 4800 5900
+Wire Wire Line
+	5050 6000 4800 6000
+Wire Wire Line
+	5050 6100 4800 6100
+Wire Wire Line
+	5950 4500 5600 4500
+Wire Wire Line
+	5950 3700 5600 3700
+Wire Wire Line
+	5950 3900 5600 3900
+Wire Wire Line
+	5950 4100 5600 4100
+Wire Wire Line
+	5950 4300 5600 4300
+Wire Wire Line
+	5950 3100 5600 3100
+Wire Wire Line
+	5950 3300 5600 3300
+Wire Wire Line
+	5950 3500 5600 3500
+Wire Wire Line
+	2600 4400 1900 4400
+Wire Wire Line
+	2250 3600 2600 3600
+Wire Wire Line
+	2600 4000 2250 4000
+Wire Wire Line
+	2600 3200 2250 3200
 $EndSCHEMATC
