File: TinyBoard84100.sch (KiCad schematic (older format))
At the start: 14 parts

Commit message: finishing schematic
Connections:
- net MISO is gone; now on net PA5: P?.1 (P1)
- net MOSI is gone; now on net PA6: P?.4 (P4)
- net SCK is gone; now on net PA4: P?.3 (P3), R?.1 (A)
- net ~RST is gone; now on net PB3: P?.5 (P5)
Other:
- note added: "+5V\n\nMOSI\n\nGND"
- note added: "MISO = PA5 (pin 8)\nMOSI = PA6 (pin 7)\nSCK/SCL = PA4 (pin 9)\n~RST~ = PB3 (pin 4)"
- note added: "MISO\n\nSCK\n\n~RST"
Changed lines of the file:
@@
 Wire Wire Line
 	9000 3350 9300 3350
-Text Label 8250 2850 0    60   ~ 0
-MISO
 Text Label 8250 3100 0    60   ~ 0
-SCK
+PA4
 Text Label 8250 3350 0    60   ~ 0
-~RST
+PB3
 Text Label 9300 3100 2    60   ~ 0
-MOSI
+PA6
 Wire Wire Line
 	10050 2800 10050 2600
@@
 	10050 2600 9850 2600
 Text Label 9850 2600 0    60   ~ 0
-SCK
+PA4
 $Comp
 L GND #PWR?
@@
 	-1   0    0    1
 $EndComp
+Text Label 8250 2850 0    60   ~ 0
+PA5
+Text Notes 8200 3300 2    60   ~ 0
+MISO\n\nSCK\n\n~RST
+Text Notes 9350 3300 0    60   ~ 0
++5V\n\nMOSI\n\nGND
+Text Notes 8100 2350 0    60   ~ 0
+MISO     = PA5 (pin 8)\nMOSI     = PA6 (pin 7)\nSCK/SCL = PA4 (pin 9)\n~RST~      = PB3 (pin 4)
 $EndSCHEMATC

Commit message: annotated & erc passed
Parts:
- C1: renamed from C?; value C -> 4.7uF
- C2: renamed from C?; value C -> 1uF
- R1, R2, R3: renamed from R?; value R -> 1k
- gave numbers to parts that had none: 9
Connections:
- net GND: now also C1.2, C2.2, P1.2 (P2), P3.1 (P1), U1.2 (GND)
- net PB3: now also SW1.2
- net at P1.1 (P1), U1.3 (IN): now also C1.1, C2.1
Other:
- moved on the sheet: D1, R3
Changed lines of the file:
@@
 $EndDescr
 $Comp
-L SW_PUSH SW?
+L SW_PUSH SW1
 U 1 1 5AD23CB0
 P 3400 4750
-F 0 "SW?" H 3550 4860 50  0000 C CNN
+F 0 "SW1" H 3550 4860 50  0000 C CNN
 F 1 "SW_PUSH" H 3400 4670 50  0000 C CNN
 F 2 "" H 3400 4750 60  0000 C CNN
@@
 $EndComp
 $Comp
-L CONN_02X03 P?
+L CONN_02X03 P4
 U 1 1 5AD23CEF
 P 8750 3100
-F 0 "P?" H 8750 3300 50  0000 C CNN
+F 0 "P4" H 8750 3300 50  0000 C CNN
 F 1 "CONN_02X03" H 8750 2900 50  0000 C CNN
 F 2 "" H 8750 1900 50  0000 C CNN
@@
 $EndComp
 $Comp
-L CONN_01X02 P?
+L CONN_01X02 P1
 U 1 1 5AD23D2C
 P 1300 1600
-F 0 "P?" H 1300 1750 50  0000 C CNN
+F 0 "P1" H 1300 1750 50  0000 C CNN
 F 1 "CONN_01X02" V 1400 1600 50  0000 C CNN
 F 2 "" H 1300 1600 50  0000 C CNN
@@
 $EndComp
 $Comp
-L R R?
+L R R1
 U 1 1 5AD23D65
 P 3000 4450
-F 0 "R?" H 3000 4525 40  0000 C CNN
-F 1 "R" H 3000 4375 40  0000 C CNN
+F 0 "R1" H 3000 4525 40  0000 C CNN
+F 1 "1k" H 3000 4375 40  0000 C CNN
 F 2 "" H 3000 4450 60  0000 C CNN
 F 3 "" H 3000 4450 60  0000 C CNN
@@
 $EndComp
 $Comp
-L R R?
+L R R3
 U 1 1 5AD23D8B
-P 10050 3000
-F 0 "R?" H 10050 3075 40  0000 C CNN
-F 1 "R" H 10050 2925 40  0000 C CNN
-F 2 "" H 10050 3000 60  0000 C CNN
-F 3 "" H 10050 3000 60  0000 C CNN
-	1    10050 3000
+P 10050 2850
+F 0 "R3" H 10050 2925 40  0000 C CNN
+F 1 "1k" H 10050 2775 40  0000 C CNN
+F 2 "" H 10050 2850 60  0000 C CNN
+F 3 "" H 10050 2850 60  0000 C CNN
+	1    10050 2850
 	0    1    1    0
 $EndComp
 $Comp
-L C C?
+L C C1
 U 1 1 5AD23DAF
 P 1850 1600
-F 0 "C?" H 1850 1700 40  0000 L CNN
-F 1 "C" H 1856 1515 40  0000 L CNN
+F 0 "C1" H 1850 1700 40  0000 L CNN
+F 1 "4.7uF" H 1856 1515 40  0000 L CNN
 F 2 "" H 1888 1450 30  0000 C CNN
 F 3 "" H 1850 1600 60  0000 C CNN
@@
 $EndComp
 $Comp
-L C C?
+L C C2
 U 1 1 5AD23DE1
 P 2100 1600
-F 0 "C?" H 2100 1700 40  0000 L CNN
-F 1 "C" H 2106 1515 40  0000 L CNN
+F 0 "C2" H 2100 1700 40  0000 L CNN
+F 1 "1uF" H 2106 1515 40  0000 L CNN
 F 2 "" H 2138 1450 30  0000 C CNN
 F 3 "" H 2100 1600 60  0000 C CNN
@@
 $EndComp
 $Comp
-L LED D?
+L LED D1
 U 1 1 5AD23E1F
-P 3200 2000
-F 0 "D?" H 3200 2100 50  0000 C CNN
-F 1 "LED" H 3200 1900 50  0000 C CNN
-F 2 "" H 3200 2000 60  0000 C CNN
-F 3 "" H 3200 2000 60  0000 C CNN
-	1    3200 2000
+P 3200 2150
+F 0 "D1" H 3200 2250 50  0000 C CNN
+F 1 "LED" H 3200 2050 50  0000 C CNN
+F 2 "" H 3200 2150 60  0000 C CNN
+F 3 "" H 3200 2150 60  0000 C CNN
+	1    3200 2150
 	0    1    1    0
 $EndComp
 $Comp
-L LED D?
+L LED D2
 U 1 1 5AD23E83
 P 10050 3400
-F 0 "D?" H 10050 3500 50  0000 C CNN
+F 0 "D2" H 10050 3500 50  0000 C CNN
 F 1 "LED" H 10050 3300 50  0000 C CNN
 F 2 "" H 10050 3400 60  0000 C CNN
@@
 $EndComp
 $Comp
-L R R?
+L R R2
 U 1 1 5AD23EBD
 P 3200 1600
-F 0 "R?" H 3200 1675 40  0000 C CNN
-F 1 "R" H 3200 1525 40  0000 C CNN
+F 0 "R2" H 3200 1675 40  0000 C CNN
+F 1 "1k" H 3200 1525 40  0000 C CNN
 F 2 "" H 3200 1600 60  0000 C CNN
 F 3 "" H 3200 1600 60  0000 C CNN
@@
 $EndComp
 $Comp
-L CONN_01X07 P?
+L CONN_01X07 P2
 U 1 1 5AD23FFE
 P 4250 5850
-F 0 "P?" H 4250 6250 50  0000 C CNN
+F 0 "P2" H 4250 6250 50  0000 C CNN
 F 1 "CONN_01X07" V 4350 5850 50  0000 C CNN
 F 2 "" H 4250 5850 50  0000 C CNN
@@
 $EndComp
 $Comp
-L CONN_01X07 P?
+L CONN_01X07 P3
 U 1 1 5AD240B6
 P 6550 5850
-F 0 "P?" H 6550 6250 50  0000 C CNN
+F 0 "P3" H 6550 6250 50  0000 C CNN
 F 1 "CONN_01X07" V 6650 5850 50  0000 C CNN
 F 2 "" H 6550 5850 50  0000 C CNN
@@
 $EndComp
 $Comp
-L PWR_FLAG #FLG?
+L PWR_FLAG #FLG01
 U 1 1 5AD2529F
 P 1700 1400
-F 0 "#FLG?" H 1700 1495 50  0001 C CNN
+F 0 "#FLG01" H 1700 1495 50  0001 C CNN
 F 1 "PWR_FLAG" H 1700 1580 50  0000 C CNN
 F 2 "" H 1700 1400 50  0000 C CNN
@@
 $EndComp
 $Comp
-L PWR_FLAG #FLG?
+L PWR_FLAG #FLG02
 U 1 1 5AD252DB
 P 1700 1800
-F 0 "#FLG?" H 1700 1895 50  0001 C CNN
+F 0 "#FLG02" H 1700 1895 50  0001 C CNN
 F 1 "PWR_FLAG" H 1700 1980 50  0000 C CNN
 F 2 "" H 1700 1800 50  0000 C CNN
@@
 $EndComp
 $Comp
-L GND #PWR?
+L GND #PWR03
 U 1 1 5AD25364
-P 2200 1800
-F 0 "#PWR?" H 2200 1550 50  0001 C CNN
-F 1 "GND" H 2200 1650 50  0000 C CNN
-F 2 "" H 2200 1800 50  0000 C CNN
-F 3 "" H 2200 1800 50  0000 C CNN
-	1    2200 1800
-	1    0    0    -1
-$EndComp
-$Comp
-L +5V #PWR?
+P 2100 1800
+F 0 "#PWR03" H 2100 1550 50  0001 C CNN
+F 1 "GND" H 2100 1650 50  0000 C CNN
+F 2 "" H 2100 1800 50  0000 C CNN
+F 3 "" H 2100 1800 50  0000 C CNN
+	1    2100 1800
+	1    0    0    -1
+$EndComp
+$Comp
+L +5V #PWR04
 U 1 1 5AD253A2
 P 3200 1300
-F 0 "#PWR?" H 3200 1150 50  0001 C CNN
+F 0 "#PWR04" H 3200 1150 50  0001 C CNN
 F 1 "+5V" H 3200 1440 50  0000 C CNN
 F 2 "" H 3200 1300 50  0000 C CNN
@@
 $EndComp
 $Comp
-L ATTINY841 U?
+L ATTINY841 U2
 U 1 1 5AD23C06
 P 5400 3850
-F 0 "U?" H 4350 4650 60  0000 C CNN
+F 0 "U2" H 4350 4650 60  0000 C CNN
 F 1 "ATTINY841" H 4500 3050 60  0000 C CNN
 F 2 "" H 6450 3250 60  0000 C CNN
@@
 	1500 1650 1500 1800
 $Comp
-L 78L05 U?
+L 78L05 U1
 U 1 1 5AD23F10
 P 2600 1500
-F 0 "U?" H 2700 1400 60  0000 C CNN
+F 0 "U1" H 2700 1400 60  0000 C CNN
 F 1 "78L05" H 2600 1750 60  0000 C CNN
 F 2 "" H 2500 1600 60  0000 C CNN
@@
 	3200 1400 3000 1400
 $Comp
-L GND #PWR?
+L GND #PWR05
 U 1 1 5AD3606C
-P 3200 2200
-F 0 "#PWR?" H 3200 1950 50  0001 C CNN
-F 1 "GND" H 3200 2050 50  0000 C CNN
-F 2 "" H 3200 2200 50  0000 C CNN
-F 3 "" H 3200 2200 50  0000 C CNN
-	1    3200 2200
+P 3200 2450
+F 0 "#PWR05" H 3200 2200 50  0001 C CNN
+F 1 "GND" H 3200 2300 50  0000 C CNN
+F 2 "" H 3200 2450 50  0000 C CNN
+F 3 "" H 3200 2450 50  0000 C CNN
+	1    3200 2450
 	1    0    0    -1
 $EndComp
@@
 	3200 1400 3200 1300
 $Comp
-L +5V #PWR?
+L +5V #PWR06
 U 1 1 5AD36244
-P 4850 2800
-F 0 "#PWR?" H 4850 2650 50  0001 C CNN
-F 1 "+5V" H 4850 2940 50  0000 C CNN
-F 2 "" H 4850 2800 50  0000 C CNN
-F 3 "" H 4850 2800 50  0000 C CNN
-	1    4850 2800
-	1    0    0    -1
-$EndComp
-$Comp
-L GND #PWR?
+P 4850 2650
+F 0 "#PWR06" H 4850 2500 50  0001 C CNN
+F 1 "+5V" H 4850 2790 50  0000 C CNN
+F 2 "" H 4850 2650 50  0000 C CNN
+F 3 "" H 4850 2650 50  0000 C CNN
+	1    4850 2650
+	1    0    0    -1
+$EndComp
+$Comp
+L GND #PWR07
 U 1 1 5AD362BF
-P 4850 4900
-F 0 "#PWR?" H 4850 4650 50  0001 C CNN
-F 1 "GND" H 4850 4750 50  0000 C CNN
-F 2 "" H 4850 4900 50  0000 C CNN
-F 3 "" H 4850 4900 50  0000 C CNN
-	1    4850 4900
-	1    0    0    -1
-$EndComp
-$Comp
-L GND #PWR?
+P 4850 5000
+F 0 "#PWR07" H 4850 4750 50  0001 C CNN
+F 1 "GND" H 4850 4850 50  0000 C CNN
+F 2 "" H 4850 5000 50  0000 C CNN
+F 3 "" H 4850 5000 50  0000 C CNN
+	1    4850 5000
+	1    0    0    -1
+$EndComp
+$Comp
+L GND #PWR08
 U 1 1 5AD36E09
 P 3400 5050
-F 0 "#PWR?" H 3400 4800 50  0001 C CNN
+F 0 "#PWR08" H 3400 4800 50  0001 C CNN
 F 1 "GND" H 3400 4900 50  0000 C CNN
 F 2 "" H 3400 5050 50  0000 C CNN
@@
 $EndComp
 $Comp
-L +5V #PWR?
+L +5V #PWR09
 U 1 1 5AD36E68
 P 2800 4300
-F 0 "#PWR?" H 2800 4150 50  0001 C CNN
+F 0 "#PWR09" H 2800 4150 50  0001 C CNN
 F 1 "+5V" H 2800 4440 50  0000 C CNN
 F 2 "" H 2800 4300 50  0000 C CNN
@@
 PA6
 Wire Wire Line
-	10050 2800 10050 2600
-Wire Wire Line
-	10050 2600 9850 2600
-Text Label 9850 2600 0    60   ~ 0
+	10050 2650 10050 2450
+Wire Wire Line
+	10050 2450 9850 2450
+Text Label 9850 2450 0    60   ~ 0
 PA4
 $Comp
-L GND #PWR?
+L GND #PWR010
 U 1 1 5AD37B93
 P 10050 3800
-F 0 "#PWR?" H 10050 3550 50  0001 C CNN
+F 0 "#PWR010" H 10050 3550 50  0001 C CNN
 F 1 "GND" H 10050 3650 50  0000 C CNN
 F 2 "" H 10050 3800 50  0000 C CNN
@@
 	10050 3800 10050 3600
 $Comp
-L GND #PWR?
+L GND #PWR011
 U 1 1 5AD37D91
 P 9300 3350
-F 0 "#PWR?" H 9300 3100 50  0001 C CNN
+F 0 "#PWR011" H 9300 3100 50  0001 C CNN
 F 1 "GND" H 9300 3200 50  0000 C CNN
 F 2 "" H 9300 3350 50  0000 C CNN
@@
 $EndComp
 $Comp
-L +5V #PWR?
+L +5V #PWR012
 U 1 1 5AD37EB4
 P 9300 2850
-F 0 "#PWR?" H 9300 2700 50  0001 C CNN
+F 0 "#PWR012" H 9300 2700 50  0001 C CNN
 F 1 "+5V" H 9300 2990 50  0000 C CNN
 F 2 "" H 9300 2850 50  0000 C CNN
@@
 	3900 3250 3550 3250
 $Comp
-L +5V #PWR?
+L +5V #PWR013
 U 1 1 5AD3A272
 P 4700 5550
-F 0 "#PWR?" H 4700 5400 50  0001 C CNN
+F 0 "#PWR013" H 4700 5400 50  0001 C CNN
 F 1 "+5V" H 4700 5690 50  0000 C CNN
 F 2 "" H 4700 5550 50  0000 C CNN
@@
 PA0
 $Comp
-L GND #PWR?
+L GND #PWR014
 U 1 1 5AD3A4E3
-P 6100 5500
-F 0 "#PWR?" H 6100 5250 50  0001 C CNN
-F 1 "GND" H 6100 5350 50  0000 C CNN
-F 2 "" H 6100 5500 50  0000 C CNN
-F 3 "" H 6100 5500 50  0000 C CNN
-	1    6100 5500
+P 6100 5550
+F 0 "#PWR014" H 6100 5300 50  0001 C CNN
+F 1 "GND" H 6100 5400 50  0000 C CNN
+F 2 "" H 6100 5550 50  0000 C CNN
+F 3 "" H 6100 5550 50  0000 C CNN
+	1    6100 5550
 	-1   0    0    1
 $EndComp
@@
 Text Notes 8100 2350 0    60   ~ 0
 MISO     = PA5 (pin 8)\nMOSI     = PA6 (pin 7)\nSCK/SCL = PA4 (pin 9)\n~RST~      = PB3 (pin 4)
+Connection ~ 1700 1400
+Connection ~ 1850 1400
+Connection ~ 2100 1400
+Connection ~ 2100 1800
+Connection ~ 1850 1800
+Connection ~ 1700 1800
+Connection ~ 3400 4450
+Wire Wire Line
+	4850 5000 4850 4900
+Wire Wire Line
+	4850 2800 4850 2650
+Wire Wire Line
+	3200 2450 3200 2350
+Wire Wire Line
+	3200 1950 3200 1800
+Wire Wire Line
+	10050 3050 10050 3200
 $EndSCHEMATC

Commit message: footprints associated
Parts:
- C1, C2: footprint (none) -> Capacitors_SMD:C_1206_HandSoldering
- D1, D2: footprint (none) -> LEDs:LED_0805
- P1: footprint (none) -> Pin_Headers:Pin_Header_Angled_1x02
- P2, P3: footprint (none) -> Pin_Headers:Pin_Header_Straight_1x07
- P4: footprint (none) -> Pin_Headers:Pin_Header_Straight_2x03
- R1, R2, R3: footprint (none) -> Resistors_SMD:R_0805_HandSoldering
- SW1: footprint (none) -> Buttons_Switches_SMD:SW_SPST_EVQPE1
- U1: footprint (none) -> TO_SOT_Packages_SMD:SOT-23_Handsoldering
- U2: footprint (none) -> Housings_SOIC:SOIC-14_3.9x8.7mm_Pitch1.27mm
Changed lines of the file:
@@
 F 0 "SW1" H 3550 4860 50  0000 C CNN
 F 1 "SW_PUSH" H 3400 4670 50  0000 C CNN
-F 2 "" H 3400 4750 60  0000 C CNN
+F 2 "Buttons_Switches_SMD:SW_SPST_EVQPE1" H 3400 4750 60  0001 C CNN
 F 3 "" H 3400 4750 60  0000 C CNN
 	1    3400 4750
@@
 F 0 "P4" H 8750 3300 50  0000 C CNN
 F 1 "CONN_02X03" H 8750 2900 50  0000 C CNN
-F 2 "" H 8750 1900 50  0000 C CNN
+F 2 "Pin_Headers:Pin_Header_Straight_2x03" H 8750 1900 50  0001 C CNN
 F 3 "" H 8750 1900 50  0000 C CNN
 	1    8750 3100
@@
 F 0 "P1" H 1300 1750 50  0000 C CNN
 F 1 "CONN_01X02" V 1400 1600 50  0000 C CNN
-F 2 "" H 1300 1600 50  0000 C CNN
+F 2 "Pin_Headers:Pin_Header_Angled_1x02" H 1300 1600 50  0001 C CNN
 F 3 "" H 1300 1600 50  0000 C CNN
 	1    1300 1600
@@
 F 0 "R1" H 3000 4525 40  0000 C CNN
 F 1 "1k" H 3000 4375 40  0000 C CNN
-F 2 "" H 3000 4450 60  0000 C CNN
+F 2 "Resistors_SMD:R_0805_HandSoldering" H 3000 4450 60  0001 C CNN
 F 3 "" H 3000 4450 60  0000 C CNN
 	1    3000 4450
@@
 F 0 "R3" H 10050 2925 40  0000 C CNN
 F 1 "1k" H 10050 2775 40  0000 C CNN
-F 2 "" H 10050 2850 60  0000 C CNN
+F 2 "Resistors_SMD:R_0805_HandSoldering" H 10050 2850 60  0001 C CNN
 F 3 "" H 10050 2850 60  0000 C CNN
 	1    10050 2850
@@
 F 0 "C1" H 1850 1700 40  0000 L CNN
 F 1 "4.7uF" H 1856 1515 40  0000 L CNN
-F 2 "" H 1888 1450 30  0000 C CNN
+F 2 "Capacitors_SMD:C_1206_HandSoldering" H 1888 1450 30  0001 C CNN
 F 3 "" H 1850 1600 60  0000 C CNN
 	1    1850 1600
@@
 F 0 "C2" H 2100 1700 40  0000 L CNN
 F 1 "1uF" H 2106 1515 40  0000 L CNN
-F 2 "" H 2138 1450 30  0000 C CNN
+F 2 "Capacitors_SMD:C_1206_HandSoldering" H 2138 1450 30  0001 C CNN
 F 3 "" H 2100 1600 60  0000 C CNN
 	1    2100 1600
@@
 F 0 "D1" H 3200 2250 50  0000 C CNN
 F 1 "LED" H 3200 2050 50  0000 C CNN
-F 2 "" H 3200 2150 60  0000 C CNN
+F 2 "LEDs:LED_0805" H 3200 2150 60  0001 C CNN
 F 3 "" H 3200 2150 60  0000 C CNN
 	1    3200 2150
@@
 F 0 "D2" H 10050 3500 50  0000 C CNN
 F 1 "LED" H 10050 3300 50  0000 C CNN
-F 2 "" H 10050 3400 60  0000 C CNN
+F 2 "LEDs:LED_0805" H 10050 3400 60  0001 C CNN
 F 3 "" H 10050 3400 60  0000 C CNN
 	1    10050 3400
@@
 F 0 "R2" H 3200 1675 40  0000 C CNN
 F 1 "1k" H 3200 1525 40  0000 C CNN
-F 2 "" H 3200 1600 60  0000 C CNN
+F 2 "Resistors_SMD:R_0805_HandSoldering" H 3200 1600 60  0001 C CNN
 F 3 "" H 3200 1600 60  0000 C CNN
 	1    3200 1600
@@
 F 0 "P2" H 4250 6250 50  0000 C CNN
 F 1 "CONN_01X07" V 4350 5850 50  0000 C CNN
-F 2 "" H 4250 5850 50  0000 C CNN
+F 2 "Pin_Headers:Pin_Header_Straight_1x07" H 4250 5850 50  0001 C CNN
 F 3 "" H 4250 5850 50  0000 C CNN
 	1    4250 5850
@@
 F 0 "P3" H 6550 6250 50  0000 C CNN
 F 1 "CONN_01X07" V 6650 5850 50  0000 C CNN
-F 2 "" H 6550 5850 50  0000 C CNN
+F 2 "Pin_Headers:Pin_Header_Straight_1x07" H 6550 5850 50  0001 C CNN
 F 3 "" H 6550 5850 50  0000 C CNN
 	1    6550 5850
@@
 F 0 "U2" H 4350 4650 60  0000 C CNN
 F 1 "ATTINY841" H 4500 3050 60  0000 C CNN
-F 2 "" H 6450 3250 60  0000 C CNN
+F 2 "Housings_SOIC:SOIC-14_3.9x8.7mm_Pitch1.27mm" H 6450 3250 60  0001 C CNN
 F 3 "" H 6450 3250 60  0000 C CNN
 	1    5400 3850
@@
 F 0 "U1" H 2700 1400 60  0000 C CNN
 F 1 "78L05" H 2600 1750 60  0000 C CNN
-F 2 "" H 2500 1600 60  0000 C CNN
+F 2 "TO_SOT_Packages_SMD:SOT-23_Handsoldering" H 2500 1600 60  0001 C CNN
 F 3 "" H 2500 1600 60  0000 C CNN
 	1    2600 1500

Commit message: corrected footprints
Parts:
- SW1: footprint Buttons_Switches_SMD:SW_SPST_EVQPE1 -> Buttons_Switches_SMD:SW_SPST_FSMSM
- U1: footprint TO_SOT_Packages_SMD:SOT-23_Handsoldering -> TO_SOT_Packages_SMD:SOT89-3_Housing_Handsoldering
Changed lines of the file:
@@
 F 0 "SW1" H 3550 4860 50  0000 C CNN
 F 1 "SW_PUSH" H 3400 4670 50  0000 C CNN
-F 2 "Buttons_Switches_SMD:SW_SPST_EVQPE1" H 3400 4750 60  0001 C CNN
+F 2 "Buttons_Switches_SMD:SW_SPST_FSMSM" H 3400 4750 60  0001 C CNN
 F 3 "" H 3400 4750 60  0000 C CNN
 	1    3400 4750
@@
 F 0 "U1" H 2700 1400 60  0000 C CNN
 F 1 "78L05" H 2600 1750 60  0000 C CNN
-F 2 "TO_SOT_Packages_SMD:SOT-23_Handsoldering" H 2500 1600 60  0001 C CNN
+F 2 "TO_SOT_Packages_SMD:SOT89-3_Housing_Handsoldering" H 2500 1600 60  0001 C CNN
 F 3 "" H 2500 1600 60  0000 C CNN
 	1    2600 1500

Commit message: corrected footprints
Parts:
- removed P1: CONN_01X02, Pin_Headers:Pin_Header_Angled_1x02, symbol CONN_01X02
Connections:
- net +5V: no longer P2.1 (P1)
- net +BATT: now reaches C1.1, C2.1, U1.3 (IN)
- net +BATT: now also P2.1 (P1)
Changed lines of the file:
@@
-$EndComp
-$Comp
-L CONN_01X02 P1
-U 1 1 5AD23D2C
-P 1300 1600
-F 0 "P1" H 1300 1750 50  0000 C CNN
-F 1 "CONN_01X02" V 1400 1600 50  0000 C CNN
-F 2 "Pin_Headers:Pin_Header_Angled_1x02" H 1300 1600 50  0001 C CNN
-F 3 "" H 1300 1600 50  0000 C CNN
-	1    1300 1600
-	-1   0    0    -1
 $EndComp
 $Comp
@@
 L PWR_FLAG #FLG02
 U 1 1 5AD252DB
-P 1700 1800
-F 0 "#FLG02" H 1700 1895 50  0001 C CNN
-F 1 "PWR_FLAG" H 1700 1980 50  0000 C CNN
-F 2 "" H 1700 1800 50  0000 C CNN
-F 3 "" H 1700 1800 50  0000 C CNN
-	1    1700 1800
+P 1500 1800
+F 0 "#FLG02" H 1500 1895 50  0001 C CNN
+F 1 "PWR_FLAG" H 1500 1980 50  0000 C CNN
+F 2 "" H 1500 1800 50  0000 C CNN
+F 3 "" H 1500 1800 50  0000 C CNN
+	1    1500 1800
 	1    0    0    1
 $EndComp
@@
 $EndComp
 Wire Wire Line
-	1500 1550 1500 1400
-Wire Wire Line
-	1500 1400 2200 1400
-Wire Wire Line
-	1500 1650 1500 1800
+	1300 1400 2200 1400
 $Comp
 L 78L05 U1
@@
 Wire Wire Line
 	3900 3250 3550 3250
-$Comp
-L +5V #PWR013
-U 1 1 5AD3A272
-P 4700 5550
-F 0 "#PWR013" H 4700 5400 50  0001 C CNN
-F 1 "+5V" H 4700 5690 50  0000 C CNN
-F 2 "" H 4700 5550 50  0000 C CNN
-F 3 "" H 4700 5550 50  0000 C CNN
-	1    4700 5550
-	1    0    0    -1
-$EndComp
 Text Label 4700 5650 2    60   ~ 0
 PB0
@@
 Connection ~ 2100 1800
 Connection ~ 1850 1800
-Connection ~ 1700 1800
 Connection ~ 3400 4450
 Wire Wire Line
@@
 Wire Wire Line
 	10050 3050 10050 3200
+$Comp
+L +BATT #PWR?
+U 1 1 5AE5D47A
+P 1300 1400
+F 0 "#PWR?" H 1300 1250 50  0001 C CNN
+F 1 "+BATT" H 1300 1540 50  0000 C CNN
+F 2 "" H 1300 1400 50  0000 C CNN
+F 3 "" H 1300 1400 50  0000 C CNN
+	1    1300 1400
+	1    0    0    -1
+$EndComp
+$Comp
+L +BATT #PWR?
+U 1 1 5AE5D609
+P 4700 5550
+F 0 "#PWR?" H 4700 5400 50  0001 C CNN
+F 1 "+BATT" H 4700 5690 50  0000 C CNN
+F 2 "" H 4700 5550 50  0000 C CNN
+F 3 "" H 4700 5550 50  0000 C CNN
+	1    4700 5550
+	1    0    0    -1
+$EndComp
 $EndSCHEMATC
