File: TinyBoard84100.kicad_pcb (KiCad board)
At the start: 2 copper layers, 27.9 x 15.2 mm, 13 parts, among them P2 CONN_01X07, P3 CONN_01X07, P4 CONN_02X03, SW1 SW_PUSH, U1 78L05, U2 ATTINY841

Commit message: finishing touches
Other:
- board text added: "."
- board text added: "ATtiny 84/841"
- board text added: "SCK"
- board text removed: "RST"
Changed lines of the file:
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@@
     (links 38)
     (no_connects 0)
-    (area 165.375 81.326666 198.405 104.093333)
+    (area 168.834999 85.014999 196.925001 100.405001)
     (thickness 1.6)
-    (drawings 27)
+    (drawings 29)
     (tracks 137)
     (zones 0)
@@
     )
   )
+  (gr_text "ATtiny\n84/841" (at 176.53 92.71) (layer F.SilkS)
+    (effects (font (size 0.9 0.9) (thickness 0.225)))
+  )
+  (gr_text . (at 172.72 93.345) (layer F.SilkS)
+    (effects (font (size 2 2) (thickness 0.5)))
+  )
   (gr_text Rev3 (at 189.865 99.695 180) (layer B.SilkS)
     (effects (font (size 0.508 0.762) (thickness 0.127)) (justify mirror))
@@
     (effects (font (size 0.762 1.016) (thickness 0.1905)) (justify mirror))
   )
-  (gr_text RST (at 195.58 95.25 180) (layer F.SilkS)
+  (gr_text SCK (at 195.58 95.25 180) (layer F.SilkS)
     (effects (font (size 0.508 0.762) (thickness 0.127)))
   )
